Commit message: First commit

File: install/ur_robotiq_description/share/ur_robotiq_description/urdf/onrobot_2fg7_upload_urdf.xacro (robot description, xacro)
@@ -124,5 +124,5 @@
   <link name="world"/>
   <joint name="world_joint" type="fixed">
-    <parent link="tool0"/>
+    <parent link="world"/>
     <child link="onrobot_2fg7_base_link"/>
     <origin rpy="0.0 0.0 0.0" xyz="0.0 0.0 0.0"/>

File: install/ur_robotiq_description/share/ur_robotiq_description/urdf/onrobot_2fg7_urdf.xacro (robot description, xacro)
@@ -1,10 +1,9 @@
 <?xml version="1.0"?>
-<!-- MAIN IDEA IS TO COPY PASTE ROBOTIQ AND REPLACE WITH 2FG7 VALUES-->
-<robot xmlns:xacro="http://wiki.ros.org/xacro" name="robotiq_gripper">
+<robot xmlns:xacro="http://wiki.ros.org/xacro" name="2fg7_outwards">
     <!-- parameters -->
     <xacro:arg name="use_fake_hardware" default="true" />
     <!-- If visualizing just the gripper with no arm, set the true, otherwise, set to false -->
     <xacro:property name="gripper_only" value="false"/>
-    <xacro:macro name="robotiq_gripper" params="
+    <xacro:macro name="2fg7_outwards" params="
         name
         prefix
@@ -17,7 +16,9 @@
         include_ros2_control:=true
         com_port:=/dev/ttyUSB0">
+        <!-- COMMENTED ROS 2 CONTROL FOR LATER -->
         <!-- ros2 control include -->
-        <xacro:include filename="$(find robotiq_description)/urdf/robotiq_gripper.ros2_control.xacro" />
+        <!-- <xacro:include filename="$(find robotiq_description)/urdf/robotiq_gripper.ros2_control.xacro" /> -->
         <!-- if we are simulating or directly communicating with the gripper we need a ros2 control instance -->
+        <!--
         <xacro:if value="${include_ros2_control}">
             <xacro:robotiq_gripper_ros2_control
@@ -29,262 +30,89 @@
                 com_port="${com_port}"/>
         </xacro:if>
-        <link name="${prefix}robotiq_85_base_link">
+        -->
+        <link name="${prefix}2fg7_base_link">
             <visual>
                 <geometry>
-                    <mesh filename="file://$(find robotiq_description)/meshes/visual/robotiq_base.dae" />
+                    <mesh filename="package://ur_robotiq_description/meshes/base_link.stl" scale="0.001 0.001 0.001"/>
                 </geometry>
             </visual>
             <collision>
                 <geometry>
-                    <mesh filename="file://$(find robotiq_description)/meshes/collision/robotiq_base.stl" />
+                    <mesh filename="package://ur_robotiq_description/meshes/base_link.stl" scale="0.001 0.001 0.001"/>
                 </geometry>
             </collision>
             <inertial>
-                <origin xyz="0.0 2.274e-05 0.03232288" rpy="0 0 0" />
-                <mass value="6.6320197e-01" />
-                <inertia ixx="5.1617816e-04" iyy="5.8802208e-04" izz="3.9462776e-04" ixy="2.936e-8" ixz="0.0" iyz="-3.2296e-7" />
+                <origin xyz="-4.898915958379213e-05 2.84756960271082e-06 0.06811082379774974" rpy="0 0 0" />
+                <mass value="1.2646523179240972"/>
+                <inertia ixx="0.001504" ixy="-0.0" ixz="-3e-06" iyy="0.001812" iyz="0.0" izz="0.001053"/>
             </inertial>
         </link>
-        <link name="${prefix}robotiq_85_left_knuckle_link">
+        <link name="${prefix}2fg7_left_finger_link">
             <visual>
                 <geometry>
-                    <mesh filename="file://$(find robotiq_description)/meshes/visual/left_knuckle.dae" />
+                    <mesh filename="package://ur_robotiq_description/meshes/base_link.stl" scale="0.001 0.001 0.001"/>
                 </geometry>
             </visual>
             <collision>
                 <geometry>
-                    <mesh filename="file://$(find robotiq_description)/meshes/collision/left_knuckle.stl" />
+                    <mesh filename="package://ur_robotiq_description/meshes/base_link.stl" scale="0.001 0.001 0.001"/>
                 </geometry>
             </collision>
             <inertial>
-                <origin xyz="0.01213197 0.0002 -0.00058647" rpy="0 0 0" />
-                <mass value="1.384773208e-02" />
-                <inertia ixx="3.5232e-7" iyy="2.31944e-6" izz="2.23136e-6" ixy="0.0" ixz="1.1744e-7" iyz="0" />
+                <origin xyz="-4.898915958379213e-05 2.84756960271082e-06 0.06811082379774974" rpy="0 0 0" />
+                <mass value="1.2646523179240972"/>
+                <inertia ixx="0.001504" ixy="-0.0" ixz="-3e-06" iyy="0.001812" iyz="0.0" izz="0.001053"/>
             </inertial>
         </link>
-        <link name="${prefix}robotiq_85_right_knuckle_link">
+        <link name="${prefix}2fg7_right_finger_link">
             <visual>
                 <geometry>
-                    <mesh filename="file://$(find robotiq_description)/meshes/visual/right_knuckle.dae" />
+                    <mesh filename="package://ur_robotiq_description/meshes/right_finger_link.stl" scale="0.001 0.001 0.001"/>
                 </geometry>
             </visual>
             <collision>
                 <geometry>
-                    <mesh filename="file://$(find robotiq_description)/meshes/collision/right_knuckle.stl" />
+                    <mesh filename="package://ur_robotiq_description/meshes/right_finger_link.stl" scale="0.001 0.001 0.001"/>
                 </geometry>
             </collision>
             <inertial>
-                <origin xyz="-0.01213197 0.0002 -0.00058647" rpy="0 0 0" />
-                <mass value="1.384773208e-02" />
-                <inertia ixx="3.5232e-7" iyy="2.31944e-6" izz="2.23136e-6" ixy="0.0" ixz="-1.1744e-7" iyz="0.0" />
+                <origin xyz="0.017874296677847158 0.02949104051991925 0.01523421548622829" rpy="0 0 0" />
+                <mass value="0.023219383355922288"/>
+                <inertia ixx="6e-06" ixy="-0.0" ixz="1e-06" iyy="5e-06" iyz="-0.0" izz="2e-06"/>
             </inertial>
         </link>
-        <link name="${prefix}robotiq_85_left_finger_link">
-            <visual>
-                <geometry>
-                    <mesh filename="file://$(find robotiq_description)/meshes/visual/left_finger.dae" />
-                </geometry>
-            </visual>
-            <collision>
-                <geometry>
-                    <mesh filename="file://$(find robotiq_description)/meshes/collision/left_finger.stl" />
-                </geometry>
-            </collision>
-            <inertial>
-                <origin xyz="0.00346899 -0.00079447 0.01867121" rpy="0 0 0" />
-                <mass value="4.260376752e-02" />
-                <inertia ixx="1.385792000000000e-05" iyy="1.183208e-05" izz="5.19672e-06" ixy="0.0" ixz="-2.17264e-06" iyz="0.0" />
-            </inertial>
-        </link>
-        <link name="${prefix}robotiq_85_right_finger_link">
-            <visual>
-                <geometry>
-                    <mesh filename="file://$(find robotiq_description)/meshes/visual/right_finger.dae" />
-                </geometry>
-            </visual>
-            <collision>
-                <geometry>
-                    <mesh filename="file://$(find robotiq_description)/meshes/collision/right_finger.stl" />
-                </geometry>
-            </collision>
-            <inertial>
-                <origin xyz="-0.00346899 -5.53e-06 0.01867121" rpy="0 0 0" />
-                <mass value="4.260376752000000e-02" />
-                <inertia ixx="1.385792e-05" iyy="1.183208e-05" izz="5.19672e-06" ixy="0.0" ixz="2.17264e-06" iyz="0.0" />
-            </inertial>
-        </link>
-        <link name="${prefix}robotiq_85_left_inner_knuckle_link">
-            <visual>
-                <geometry>
-                    <mesh filename="file://$(find robotiq_description)/meshes/visual/left_inner_knuckle.dae" />
-                </geometry>
-            </visual>
-            <collision>
-                <geometry>
-                    <mesh filename="file://$(find robotiq_description)/meshes/collision/left_inner_knuckle.stl" />
-                </geometry>
-            </collision>
-            <inertial>
-                <origin xyz="0.01897699 0.00015001 0.02247101" rpy="0 0 0" />
-                <mass value="2.969376448e-02" />
-                <inertia ixx="9.57136e-06" iyy="8.69056e-06" izz="8.19144e-06" ixy="0.0" ixz="-3.93424e-06" iyz="0.0" />
-            </inertial>
-        </link>
-        <link name="${prefix}robotiq_85_right_inner_knuckle_link">
-            <visual>
-                <geometry>
-                    <mesh filename="file://$(find robotiq_description)/meshes/visual/right_inner_knuckle.dae" />
-                </geometry>
-            </visual>
-            <collision>
-                <geometry>
-                    <mesh filename="file://$(find robotiq_description)/meshes/collision/right_inner_knuckle.stl" />
-                </geometry>
-            </collision>
-            <inertial>
-                <origin xyz="-0.01926824 5.001e-05 0.02222178" rpy="0 0 0" />
-                <mass value="2.969376448e-02" />
-                <inertia ixx="9.42456e-06" iyy="8.69056e-06" izz="8.33824e-06" ixy="0.0" ixz="3.9636e-06" iyz="0.0" />
-            </inertial>
-        </link>
-        <link name="${prefix}robotiq_85_left_finger_tip_link">
-            <visual>
-                <geometry>
-                    <mesh filename="file://$(find robotiq_description)/meshes/visual/left_finger_tip.dae" />
-                </geometry>
-            </visual>
-            <collision>
-                <geometry>
-                    <mesh filename="file://$(find robotiq_description)/meshes/collision/left_finger_tip.stl" />
-                </geometry>
-                <surface>
-                    <friction>
-                    <ode>
-                        <mu1>100000.0</mu1>
-                        <mu2>100000.0</mu2>
-                    </ode>
-                    </friction>
-                    <contact>
-                    <ode>
-                        <kp>1e+5</kp>
-                        <kd>1</kd>
-                        <soft_cfm>0</soft_cfm>
-                        <soft_erp>0.2</soft_erp>
-                        <minDepth>0.002</minDepth>
-                        <maxVel>0</maxVel>
-                    </ode>
-                    </contact>
-                </surface>
-            </collision>
-            <inertial>
-                <origin xyz="-0.01456706 -0.0008 0.01649701" rpy="0 0 0" />
-                <mass value="4.268588744e-02" />
-                <inertia ixx="1.048152e-05" iyy="1.197888e-05" izz="4.22784e-06" ixy="0.0" ixz="3.5232e-6" iyz="0.0" />
-            </inertial>
-        </link>
-        <link name="${prefix}robotiq_85_right_finger_tip_link">
-            <visual>
-                <geometry>
-                    <mesh filename="file://$(find robotiq_description)/meshes/visual/right_finger_tip.dae" />
-                </geometry>
-            </visual>
-            <collision>
-                <geometry>
-                    <mesh filename="file://$(find robotiq_description)/meshes/collision/right_finger_tip.stl" />
-                </geometry>
-                <surface>
-                    <friction>
-                    <ode>
-                        <mu1>100000.0</mu1>
-                        <mu2>100000.0</mu2>
-                    </ode>
-                    </friction>
-                    <contact>
-                    <ode>
-                        <kp>1e+5</kp>
-                        <kd>1</kd>
-                        <soft_cfm>0</soft_cfm>
-                        <soft_erp>0.2</soft_erp>
-                        <minDepth>0.002</minDepth>
-                        <maxVel>0</maxVel>
-                    </ode>
-                    </contact>
-                </surface>
-            </collision>
-            <inertial>
-                <origin xyz="0.01456706 5e-05 0.01649701" rpy="0 0 0" />
-                <mass value="4.268588744e-02" />
-                <inertia ixx="1.048152e-05" iyy="1.197888e-05" izz="4.22784e-06" ixy="0.0" ixz="-3.5232e-06" iyz="0.0" />
-            </inertial>
-        </link>
-        <joint name="${prefix}robotiq_85_base_joint" type="fixed">
-            <parent link="${parent}" />
-            <child link="${prefix}robotiq_85_base_link" />
+        <joint name="${prefix}2fg7_base_joint" type="fixed">
+            <parent link="tool0" />
+            <child link="${prefix}2fg7_base_link" />
             <xacro:insert_block name="origin" />
         </joint>
-        <joint name="${prefix}robotiq_85_left_knuckle_joint" type="revolute">
-            <parent link="${prefix}robotiq_85_base_link" />
-            <child link="${prefix}robotiq_85_left_knuckle_link" />
-            <axis xyz="0 -1 0" />
-            <origin xyz="0.03060114 0.0 0.05490452" rpy="0 0 0" />
-            <limit lower="0.0" upper="0.8" velocity="0.5" effort="50" />
+        <joint name="${prefix}2fg7_left_finger_joint" type="prismatic">
+            <parent link="${prefix}2fg7_base_link" />
+            <child link="${prefix}2fg7_left_finger_link" />
+            <axis xyz="-1 0 0" />
+            <origin xyz="0.032239 -0.029494 0.12005" rpy="0 0 0" />
+            <limit lower="0.0" upper="0.019" velocity="0.45" effort="140" />
         </joint>
-        <joint name="${prefix}robotiq_85_right_knuckle_joint" type="revolute">
-            <parent link="${prefix}robotiq_85_base_link" />
-            <child link="${prefix}robotiq_85_right_knuckle_link" />
-            <axis xyz="0 -1 0" />
-            <origin xyz="-0.03060114 0.0 0.05490452" rpy="0 0 0" />
-            <limit lower="-0.8" upper="0.0" velocity="0.5" effort="50" />
-            <mimic joint="${prefix}robotiq_85_left_knuckle_joint" multiplier="-1" />
-        </joint>
-        <joint name="${prefix}robotiq_85_left_finger_joint" type="fixed">
-            <parent link="${prefix}robotiq_85_left_knuckle_link" />
-            <child link="${prefix}robotiq_85_left_finger_link" />
-            <origin xyz="0.03152616 0.0 -0.00376347" rpy="0 0 0" />
-        </joint>
-        <joint name="${prefix}robotiq_85_right_finger_joint" type="fixed">
-            <parent link="${prefix}robotiq_85_right_knuckle_link" />
-            <child link="${prefix}robotiq_85_right_finger_link" />
-            <origin xyz="-0.03152616 0.0 -0.00376347" rpy="0 0 0" />
-        </joint>
-        <joint name="${prefix}robotiq_85_left_inner_knuckle_joint" type="continuous">
-            <parent link="${prefix}robotiq_85_base_link" />
-            <child link="${prefix}robotiq_85_left_inner_knuckle_link" />
-            <axis xyz="0 -1 0" />
-            <origin xyz="0.0127 0.0 0.06142" rpy="0 0 0" />
-            <mimic joint="${prefix}robotiq_85_left_knuckle_joint" />
-        </joint>
-        <joint name="${prefix}robotiq_85_right_inner_knuckle_joint" type="continuous">
-            <parent link="${prefix}robotiq_85_base_link" />
-            <child link="${prefix}robotiq_85_right_inner_knuckle_link" />
-            <axis xyz="0 -1 0" />
-            <origin xyz="-0.0127 0.0 0.06142" rpy="0 0 0" />
-            <mimic joint="${prefix}robotiq_85_left_knuckle_joint" multiplier="-1" />
-        </joint>
-        <joint name="${prefix}robotiq_85_left_finger_tip_joint" type="continuous">
-            <parent link="${prefix}robotiq_85_left_finger_link" />
-            <child link="${prefix}robotiq_85_left_finger_tip_link" />
-            <axis xyz="0 -1 0" />
-            <origin xyz="0.00563134 0.0 0.04718515" rpy="0 0 0" />
-            <mimic joint="${prefix}robotiq_85_left_knuckle_joint" multiplier="-1" />
-        </joint>
-        <joint name="${prefix}robotiq_85_right_finger_tip_joint" type="continuous">
-            <parent link="${prefix}robotiq_85_right_finger_link" />
-            <child link="${prefix}robotiq_85_right_finger_tip_link" />
-            <axis xyz="0 -1 0" />
-            <origin xyz="-0.00563134 0.0 0.04718515" rpy="0 0 0" />
-            <mimic joint="${prefix}robotiq_85_left_knuckle_joint" />
+        <joint name="${prefix}2fg7_right_finger_joint" type="prismatic">
+            <parent link="${prefix}2fg7_base_link" />
+            <child link="${prefix}2fg7_right_finger_link" />
+            <axis xyz="1 0 0" />
+            <origin xyz="-0.054361 -0.029494 0.12005" rpy="0 0 0" />
+            <limit lower="-0.019" upper="0.019" velocity="0.45" effort="140" />
+            <mimic joint="2fg7_left_finger_joint" multiplier="1.0"/>
         </joint>
     </xacro:macro>
+    <!--
     <xacro:if value="${gripper_only}">
     	<link name="base_link" />
-    	<xacro:robotiq_gripper name="RobotiqGripperHardwareInterface" prefix="" parent="base_link" use_fake_hardware="$(arg use_fake_hardware)">
+    	<xacro:2fg7_outwards name="Onrobot2FG7GripperHardwareInterface" prefix="" parent="base_link" use_fake_hardware="$(arg use_fake_hardware)">
         	<origin xyz="0 0 0" rpy="0 0 0" />
-    	</xacro:robotiq_gripper>
+    	</xacro:2fg7_outwards>
     </xacro:if>
     <xacro:if value="${not gripper_only}">
-    	<xacro:robotiq_gripper name="RobotiqGripperHardwareInterface" prefix="" parent="tool0" use_fake_hardware="$(arg use_fake_hardware)">
+    	<xacro:2fg7_outwards name="Onrobot2FG7GripperHardwareInterface" prefix="" parent="tool0" use_fake_hardware="$(arg use_fake_hardware)">
         	<origin xyz="0 0 0" rpy="0 0 0" />
-    	</xacro:robotiq_gripper>
+    	</xacro:2fg7_outwards>
     </xacro:if>
+    -->
 </robot>
