Commit message: RViz UR3e and gripper 2FG7

File: install/ur_robotiq_description/share/ur_robotiq_description/urdf/onrobot_2fg7_upload_urdf.xacro (robot description, xacro)
@@ -8,5 +8,6 @@
     <color rgba="0.700 0.700 0.700 1.000"/>
   </material>
-  <gazebo reference="gripper_base_link">
+  <!--
+  <gazebo reference="onrobot_2fg7_base_link">
     <material>Gazebo/Grey</material>
     <implicitSpringDamper>1</implicitSpringDamper>
@@ -46,4 +47,5 @@
     </actuator>
   </transmission>
+  -->
   <link name="onrobot_2fg7_base_link">
     <inertial>
@@ -122,10 +124,11 @@
     <mimic joint="left_finger_joint" multiplier="1.0"/>
   </joint>
-  <link name="world"/>
+  <!-- <link name="base_link"/> -->
   <joint name="world_joint" type="fixed">
-    <parent link="world"/>
+    <parent link="tool0"/>
     <child link="onrobot_2fg7_base_link"/>
     <origin rpy="0.0 0.0 0.0" xyz="0.0 0.0 0.0"/>
   </joint>
+  <!--
   <gazebo>
     <plugin filename="libgazebo_grasp_fix.so" name="gazebo_grasp_fix">
@@ -145,12 +148,15 @@
     </plugin>
   </gazebo>
+  -->
+  <!-- loading plugin: mimic joints works in gazebo now -->
+  <!-- AFTER mimicJOint: <multiplier>1.0</multiplier>
+                <offset>0.0</offset -->
+  <!--
   <gazebo>
-    <!-- loading plugin: mimic joints works in gazebo now -->
     <plugin filename="libroboticsgroup_upatras_gazebo_mimic_joint_plugin.so" name="mimic_2FG7">
       <joint>left_finger_joint</joint>
       <mimicJoint>right_finger_joint</mimicJoint>
-      <!--multiplier>1.0</multiplier>
-              <offset>0.0</offset-->
     </plugin>
   </gazebo>
+  -->
 </robot>

File: install/ur_robotiq_description/share/ur_robotiq_description/urdf/onrobot_2fg7_urdf.xacro (robot description, xacro)
@@ -4,5 +4,5 @@
     <xacro:arg name="use_fake_hardware" default="true" />
     <!-- If visualizing just the gripper with no arm, set the true, otherwise, set to false -->
-    <xacro:property name="gripper_only" value="false"/>
+    <xacro:property name="gripper_only" value="true"/>
     <xacro:macro name="2fg7_outwards" params="
         name
@@ -16,11 +16,12 @@
         include_ros2_control:=true
         com_port:=/dev/ttyUSB0">
-        <!-- COMMENTED ROS 2 CONTROL FOR LATER -->
         <!-- ros2 control include -->
-        <!-- <xacro:include filename="$(find robotiq_description)/urdf/robotiq_gripper.ros2_control.xacro" /> -->
+        <!--
+        <xacro:include filename="package://ur_robotiq_description/urdf/onrobot_2fg7_gripper.ros2_control.xacro" />
+        -->
         <!-- if we are simulating or directly communicating with the gripper we need a ros2 control instance -->
         <!--
         <xacro:if value="${include_ros2_control}">
-            <xacro:robotiq_gripper_ros2_control
+            <xacro:onrobot_2fg7_gripper_ros2_control
                 name="${name}" prefix="${prefix}"
                 sim_ignition="${sim_ignition}"
@@ -83,5 +84,5 @@
         </link>
         <joint name="${prefix}2fg7_base_joint" type="fixed">
-            <parent link="tool0" />
+            <parent link="base_link" />
             <child link="${prefix}2fg7_base_link" />
             <xacro:insert_block name="origin" />

File: install/ur_robotiq_description/share/ur_robotiq_description/urdf/ur3e_robotiq_2f_85_urdf.xacro (robot description, xacro)
@@ -5,4 +5,4 @@
     <!-- Include macros for the UR3e and the Robotiq 2f-85 gripper -->
     <xacro:include filename="$(find ur_robotiq_description)/urdf/ur3e_urdf.xacro" />
-    <xacro:include filename="$(find ur_robotiq_description)/urdf/onrobot_2fg7_urdf.xacro" />
+    <xacro:include filename="$(find ur_robotiq_description)/urdf/robotiq_2f_85_urdf.xacro" />
 </robot>

File: src/ur_robotiq/ur_robotiq_description/urdf/onrobot_2fg7_urdf.xacro (robot description, xacro)
@@ -1,118 +1,162 @@
-<?xml version="1.0"?>
-<robot xmlns:xacro="http://wiki.ros.org/xacro" name="2fg7_outwards">
-    <!-- parameters -->
-    <xacro:arg name="use_fake_hardware" default="true" />
-    <!-- If visualizing just the gripper with no arm, set the true, otherwise, set to false -->
-    <xacro:property name="gripper_only" value="false"/>
-    <xacro:macro name="2fg7_outwards" params="
-        name
-        prefix
-        parent
-        *origin
-        sim_ignition:=false
-        sim_isaac:=false
-        use_fake_hardware:=false
-        fake_sensor_commands:=false
-        include_ros2_control:=true
-        com_port:=/dev/ttyUSB0">
-        <!-- COMMENTED ROS 2 CONTROL FOR LATER -->
-        <!-- ros2 control include -->
-        <!-- <xacro:include filename="$(find robotiq_description)/urdf/robotiq_gripper.ros2_control.xacro" /> -->
-        <!-- if we are simulating or directly communicating with the gripper we need a ros2 control instance -->
-        <!--
-        <xacro:if value="${include_ros2_control}">
-            <xacro:robotiq_gripper_ros2_control
-                name="${name}" prefix="${prefix}"
-                sim_ignition="${sim_ignition}"
-                sim_isaac="${sim_isaac}"
-                use_fake_hardware="${use_fake_hardware}"
-                fake_sensor_commands="${fake_sensor_commands}"
-                com_port="${com_port}"/>
-        </xacro:if>
-        -->
-        <link name="${prefix}2fg7_base_link">
-            <visual>
-                <geometry>
-                    <mesh filename="package://ur_robotiq_description/meshes/base_link.stl" scale="0.001 0.001 0.001"/>
-                </geometry>
-            </visual>
-            <collision>
-                <geometry>
-                    <mesh filename="package://ur_robotiq_description/meshes/base_link.stl" scale="0.001 0.001 0.001"/>
-                </geometry>
-            </collision>
-            <inertial>
-                <origin xyz="-4.898915958379213e-05 2.84756960271082e-06 0.06811082379774974" rpy="0 0 0" />
-                <mass value="1.2646523179240972"/>
-                <inertia ixx="0.001504" ixy="-0.0" ixz="-3e-06" iyy="0.001812" iyz="0.0" izz="0.001053"/>
-            </inertial>
-        </link>
-        <link name="${prefix}2fg7_left_finger_link">
-            <visual>
-                <geometry>
-                    <mesh filename="package://ur_robotiq_description/meshes/base_link.stl" scale="0.001 0.001 0.001"/>
-                </geometry>
-            </visual>
-            <collision>
-                <geometry>
-                    <mesh filename="package://ur_robotiq_description/meshes/base_link.stl" scale="0.001 0.001 0.001"/>
-                </geometry>
-            </collision>
-            <inertial>
-                <origin xyz="-4.898915958379213e-05 2.84756960271082e-06 0.06811082379774974" rpy="0 0 0" />
-                <mass value="1.2646523179240972"/>
-                <inertia ixx="0.001504" ixy="-0.0" ixz="-3e-06" iyy="0.001812" iyz="0.0" izz="0.001053"/>
-            </inertial>
-        </link>
-        <link name="${prefix}2fg7_right_finger_link">
-            <visual>
-                <geometry>
-                    <mesh filename="package://ur_robotiq_description/meshes/right_finger_link.stl" scale="0.001 0.001 0.001"/>
-                </geometry>
-            </visual>
-            <collision>
-                <geometry>
-                    <mesh filename="package://ur_robotiq_description/meshes/right_finger_link.stl" scale="0.001 0.001 0.001"/>
-                </geometry>
-            </collision>
-            <inertial>
-                <origin xyz="0.017874296677847158 0.02949104051991925 0.01523421548622829" rpy="0 0 0" />
-                <mass value="0.023219383355922288"/>
-                <inertia ixx="6e-06" ixy="-0.0" ixz="1e-06" iyy="5e-06" iyz="-0.0" izz="2e-06"/>
-            </inertial>
-        </link>
-        <joint name="${prefix}2fg7_base_joint" type="fixed">
-            <parent link="tool0" />
-            <child link="${prefix}2fg7_base_link" />
-            <xacro:insert_block name="origin" />
-        </joint>
-        <joint name="${prefix}2fg7_left_finger_joint" type="prismatic">
-            <parent link="${prefix}2fg7_base_link" />
-            <child link="${prefix}2fg7_left_finger_link" />
-            <axis xyz="-1 0 0" />
-            <origin xyz="0.032239 -0.029494 0.12005" rpy="0 0 0" />
-            <limit lower="0.0" upper="0.019" velocity="0.45" effort="140" />
-        </joint>
-        <joint name="${prefix}2fg7_right_finger_joint" type="prismatic">
-            <parent link="${prefix}2fg7_base_link" />
-            <child link="${prefix}2fg7_right_finger_link" />
-            <axis xyz="1 0 0" />
-            <origin xyz="-0.054361 -0.029494 0.12005" rpy="0 0 0" />
-            <limit lower="-0.019" upper="0.019" velocity="0.45" effort="140" />
-            <mimic joint="2fg7_left_finger_joint" multiplier="1.0"/>
-        </joint>
-    </xacro:macro>
-    <!--
-    <xacro:if value="${gripper_only}">
-    	<link name="base_link" />
-    	<xacro:2fg7_outwards name="Onrobot2FG7GripperHardwareInterface" prefix="" parent="base_link" use_fake_hardware="$(arg use_fake_hardware)">
-        	<origin xyz="0 0 0" rpy="0 0 0" />
-    	</xacro:2fg7_outwards>
-    </xacro:if>
-    <xacro:if value="${not gripper_only}">
-    	<xacro:2fg7_outwards name="Onrobot2FG7GripperHardwareInterface" prefix="" parent="tool0" use_fake_hardware="$(arg use_fake_hardware)">
-        	<origin xyz="0 0 0" rpy="0 0 0" />
-    	</xacro:2fg7_outwards>
-    </xacro:if>
-    -->
+<?xml version="1.0" ?>
+<!-- =================================================================================== -->
+<!-- |    This document was autogenerated by xacro from urdf/onrobot_2fg7_upload.xacro | -->
+<!-- |    EDITING THIS FILE BY HAND IS NOT RECOMMENDED                                 | -->
+<!-- =================================================================================== -->
+<robot name="2fg7_outwards">
+  <material name="silver">
+    <color rgba="0.700 0.700 0.700 1.000"/>
+  </material>
+  <!--
+  <gazebo reference="onrobot_2fg7_base_link">
+    <material>Gazebo/Grey</material>
+    <implicitSpringDamper>1</implicitSpringDamper>
+    <mu1>0.2</mu1>
+    <mu2>0.2</mu2>
+    <kp>100000000.0</kp>
+    <kd>1.0</kd>
+    <selfCollide>true</selfCollide>
+    <gravity>true</gravity>
+  </gazebo>
+  <gazebo reference="right_finger_link">
+    <material>Gazebo/Grey</material>
+    <implicitSpringDamper>1</implicitSpringDamper>
+    <mu1>0.2</mu1>
+    <mu2>0.2</mu2>
+    <kp>100000000.0</kp>
+    <kd>1.0</kd>
+    <selfCollide>true</selfCollide>
+  </gazebo>
+  <gazebo reference="left_finger_link">
+    <material>Gazebo/Grey</material>
+    <implicitSpringDamper>1</implicitSpringDamper>
+    <mu1>0.2</mu1>
+    <mu2>0.2</mu2>
+    <kp>100000000.0</kp>
+    <kd>1.0</kd>
+    <selfCollide>true</selfCollide>
+  </gazebo>
+  <transmission name="left_finger_joint_tran">
+    <type>transmission_interface/SimpleTransmission</type>
+    <joint name="left_finger_joint">
+      <hardwareInterface>hardware_interface/PositionJointInterface</hardwareInterface>
+    </joint>
+    <actuator name="left_finger_joint_motor">
+      <hardwareInterface>hardware_interface/PositionJointInterface</hardwareInterface>
+      <mechanicalReduction>1</mechanicalReduction>
+    </actuator>
+  </transmission>
+  -->
+  <link name="onrobot_2fg7_base_link">
+    <inertial>
+      <origin rpy="0 0 0" xyz="-4.898915958379213e-05 2.84756960271082e-06 0.06811082379774974"/>
+      <mass value="1.2646523179240972"/>
+      <inertia ixx="0.001504" ixy="-0.0" ixz="-3e-06" iyy="0.001812" iyz="0.0" izz="0.001053"/>
+    </inertial>
+    <visual>
+      <origin rpy="0 0 0" xyz="0 0 0"/>
+      <geometry>
+        <mesh filename="package://ur_robotiq_description/meshes/base_link.stl" scale="0.001 0.001 0.001"/>
+      </geometry>
+      <material name="silver"/>
+    </visual>
+    <collision>
+      <origin rpy="0 0 0" xyz="0 0 0"/>
+      <geometry>
+        <mesh filename="package://ur_robotiq_description/meshes/base_link.stl" scale="0.001 0.001 0.001"/>
+      </geometry>
+    </collision>
+  </link>
+  <link name="right_finger_link">
+    <inertial>
+      <origin rpy="0 0 0" xyz="0.017874296677847158 0.02949104051991925 0.01523421548622829"/>
+      <mass value="0.023219383355922288"/>
+      <inertia ixx="6e-06" ixy="-0.0" ixz="1e-06" iyy="5e-06" iyz="-0.0" izz="2e-06"/>
+    </inertial>
+    <visual>
+      <origin rpy="0 0 0" xyz="0.054361 0.029494 -0.12005"/>
+      <geometry>
+        <mesh filename="package://ur_robotiq_description/meshes/right_finger_link.stl" scale="0.001 0.001 0.001"/>
+      </geometry>
+      <material name="silver"/>
+    </visual>
+    <collision name="right_finger_collision">
+      <origin rpy="0 0 0" xyz="0.054361 0.029494 -0.12005"/>
+      <geometry>
+        <mesh filename="package://ur_robotiq_description/meshes/right_finger_link.stl" scale="0.001 0.001 0.001"/>
+      </geometry>
+    </collision>
+  </link>
+  <link name="left_finger_link">
+    <inertial>
+      <origin rpy="0 0 0" xyz="0.004247703322119739 0.029496959480080673 0.015234215486237948"/>
+      <mass value="0.023219383355922288"/>
+      <inertia ixx="6e-06" ixy="-0.0" ixz="-1e-06" iyy="5e-06" iyz="0.0" izz="2e-06"/>
+    </inertial>
+    <visual>
+      <origin rpy="0 0 0" xyz="-0.032239 0.029494 -0.12005"/>
+      <geometry>
+        <mesh filename="package://ur_robotiq_description/meshes/left_finger_link.stl" scale="0.001 0.001 0.001"/>
+      </geometry>
+      <material name="silver"/>
+    </visual>
+    <collision name="left_finger_collision">
+      <origin rpy="0 0 0" xyz="-0.032239 0.029494 -0.12005"/>
+      <geometry>
+        <mesh filename="package://ur_robotiq_description/meshes/left_finger_link.stl" scale="0.001 0.001 0.001"/>
+      </geometry>
+    </collision>
+  </link>
+  <joint name="left_finger_joint" type="prismatic">
+    <origin rpy="0 0 0" xyz="0.032239 -0.029494 0.12005"/>
+    <parent link="onrobot_2fg7_base_link"/>
+    <child link="left_finger_link"/>
+    <axis xyz="-1.0 0.0 0.0"/>
+    <limit effort="140" lower="0.0" upper="0.019" velocity="0.45"/>
+    <!-- total 0.38 -->
+  </joint>
+  <joint name="right_finger_joint" type="prismatic">
+    <origin rpy="0 0 0" xyz="-0.054361 -0.029494 0.12005"/>
+    <parent link="onrobot_2fg7_base_link"/>
+    <child link="right_finger_link"/>
+    <axis xyz="1.0 0.0 0.0"/>
+    <limit effort="140" lower="-0.019" upper="0.019" velocity="0.45"/>
+    <mimic joint="left_finger_joint" multiplier="1.0"/>
+  </joint>
+  <!-- <link name="base_link"/> -->
+  <joint name="world_joint" type="fixed">
+    <parent link="tool0"/>
+    <child link="onrobot_2fg7_base_link"/>
+    <origin rpy="0.0 0.0 0.0" xyz="0.0 0.0 0.0"/>
+  </joint>
+  <!--
+  <gazebo>
+    <plugin filename="libgazebo_grasp_fix.so" name="gazebo_grasp_fix">
+      <arm>
+        <arm_name>2FG7</arm_name>
+        <palm_link>onrobot_2fg7_base_link</palm_link>
+        <gripper_link>left_finger_link</gripper_link>
+        <gripper_link>right_finger_link</gripper_link>
+      </arm>
+      <forces_angle_tolerance>80</forces_angle_tolerance>
+      <update_rate>10</update_rate>
+      <grip_count_threshold>1</grip_count_threshold>
+      <max_grip_count>3</max_grip_count>
+      <release_tolerance>0.01</release_tolerance>
+      <disable_collisions_on_attach>false</disable_collisions_on_attach>
+      <contact_topic>__default_topic__</contact_topic>
+    </plugin>
+  </gazebo>
+  -->
+  <!-- loading plugin: mimic joints works in gazebo now -->
+  <!-- AFTER mimicJOint: <multiplier>1.0</multiplier>
+                <offset>0.0</offset -->
+  <!--
+  <gazebo>
+    <plugin filename="libroboticsgroup_upatras_gazebo_mimic_joint_plugin.so" name="mimic_2FG7">
+      <joint>left_finger_joint</joint>
+      <mimicJoint>right_finger_joint</mimicJoint>
+    </plugin>
+  </gazebo>
+  -->
 </robot>

File: src/ur_robotiq/ur_robotiq_description/urdf/ur3e_onrobot_2fg7_urdf.xacro (robot description, xacro)
@@ -2,7 +2,7 @@
 <robot xmlns:xacro="http://wiki.ros.org/xacro" name="ur3e_robotiq">
 	<!-- This xacro file combines the UR3e collaborative robotic arm and the
-		Robotiq 2F-85 gripper. -->
-    <!-- Include macros for the UR3e and the Robotiq 2f-85 gripper -->
+		OnRobot 2FG7 gripper. -->
+    <!-- Include macros for the UR3e and the OnRobot 2FG7 gripper -->
     <xacro:include filename="$(find ur_robotiq_description)/urdf/ur3e_urdf.xacro" />
-    <xacro:include filename="$(find ur_robotiq_description)/urdf/robotiq_2f_85_urdf.xacro" />
+    <xacro:include filename="$(find ur_robotiq_description)/urdf/onrobot_2fg7_upload_urdf.xacro" />
 </robot>
