Commit message: Fixing Gazebo

File: src/ur_custom/ur_custom_description/sdf_src/ur3e_onrobot_2fg7.urdf (robot description, URDF)
Before this commit: robot ur3e_robot, 11 links, 10 joints
Links:
- added link l515_base, mass 0.1; collision cylinder length=0.04 radius=0.03; visual cylinder length=0.04 radius=0.03
- added link left_finger_link, mass 0.023219383355922288; collision mesh filename=package://ur_custom_description/meshes/left_finger_link.stl scale=0.001 0.001 0.001; visual mesh filename=package://ur_custom_description/meshes/left_finger_link.stl scale=0.001 0.001 0.001
- added link onrobot_2fg7_base_link, mass 1.2646523179240972; collision mesh filename=package://ur_custom_description/meshes/base_link.stl scale=0.001 0.001 0.001; visual mesh filename=package://ur_custom_description/meshes/base_link.stl scale=0.001 0.001 0.001
- added link right_finger_link, mass 0.023219383355922288; collision mesh filename=package://ur_custom_description/meshes/right_finger_link.stl scale=0.001 0.001 0.001; visual mesh filename=package://ur_custom_description/meshes/right_finger_link.stl scale=0.001 0.001 0.001
Joints:
- added joint gripper_to_l515: type fixed, parent tool0, child l515_base, origin xyz=0 0 0 rpy=0 0 0
- added joint left_finger_joint: type prismatic, parent onrobot_2fg7_base_link, child left_finger_link, origin xyz=0.032239 -0.029494 0.12005 rpy=0 0 0, axis -1.0 0.0 0.0, limit lower=0.0 upper=0.019 effort=140 velocity=0.45
- added joint right_finger_joint: type prismatic, parent onrobot_2fg7_base_link, child right_finger_link, origin xyz=-0.054361 -0.029494 0.12005 rpy=0 0 0, axis 1.0 0.0 0.0, limit lower=-0.019 upper=0.019 effort=140 velocity=0.45, mimic joint=left_finger_joint multiplier=1.0
- added joint world_joint: type fixed, parent tool0, child onrobot_2fg7_base_link, origin xyz=0.0 0.0 0.0 rpy=0.0 0.0 0.0

File: src/ur_custom/ur_custom_description/urdf/onrobot_2fg7_urdf.xacro (robot description, xacro)
@@ -4,5 +4,4 @@
     <color rgba="0.700 0.700 0.700 1.000"/>
   </material>
-  <!--
   <gazebo reference="onrobot_2fg7_base_link">
     <material>Gazebo/Grey</material>
@@ -33,4 +32,5 @@
     <selfCollide>true</selfCollide>
   </gazebo>
+  <!--
   <transmission name="left_finger_joint_tran">
     <type>transmission_interface/SimpleTransmission</type>
@@ -126,5 +126,4 @@
     <origin rpy="0.0 0.0 0.0" xyz="0.0 0.0 0.0"/>
   </joint>
-  <!--
   <gazebo>
     <plugin filename="libgazebo_grasp_fix.so" name="gazebo_grasp_fix">
@@ -144,15 +143,12 @@
     </plugin>
   </gazebo>
-  -->
   <!-- loading plugin: mimic joints works in gazebo now -->
-  <!-- AFTER mimicJOint: <multiplier>1.0</multiplier>
-                <offset>0.0</offset -->
-  <!--
   <gazebo>
     <plugin filename="libroboticsgroup_upatras_gazebo_mimic_joint_plugin.so" name="mimic_2FG7">
       <joint>left_finger_joint</joint>
       <mimicJoint>right_finger_joint</mimicJoint>
+      <multiplier>1.0</multiplier>
+      <offset>0.0</offset>
     </plugin>
   </gazebo>
-  -->
 </robot>

File: src/ur_custom/ur_custom_description/urdf/realsense_L515_urdf.xacro (robot description, xacro)
@@ -1,4 +1,27 @@
 <?xml version="1.0" ?>
 <robot name="realsense_L515_camera">
+  <gazebo reference="l515_camera_link">
+    <sensor name="l515_camera" type="camera">
+      <camera>
+        <horizontal_fov>1.047</horizontal_fov> <!-- 60 degrees -->
+        <image>
+          <width>1280</width>
+          <height>720</height>
+          <format>R8G8B8</format>
+        </image>
+        <clip>
+          <near>0.1</near>
+          <far>100.0</far>
+        </clip>
+      </camera>
+      <plugin name="camera_controller" filename="gz-sim-camera-system">
+        <ros>
+          <namespace>/l515</namespace>
+          <remapping>image_raw:=image_raw</remapping>
+          <remapping>camera_info:=camera_info</remapping>
+        </ros>
+      </plugin>
+    </sensor>
+  </gazebo>
   <link name="l515_base">
     <visual>

File: src/ur_custom/ur_custom_description/urdf/ur3e_onrobot_2fg7_urdf.xacro (robot description, xacro)
@@ -1,9 +1,16 @@
 <?xml version="1.0"?>
-<robot xmlns:xacro="http://wiki.ros.org/xacro" name="ur3e_robotiq">
+<robot xmlns:xacro="http://wiki.ros.org/xacro" name="ur3e_2fg7_l515">
 	<!-- This xacro file combines the UR3e collaborative robotic arm, the
 		OnRobot 2FG7 gripper and a simplified version of the Realsense L515 Camera. -->
+    <!-- Gazebo plugin for ROS 2 joint control-->
+	<gazebo>
+      <plugin name="gz_ros2_control" filename="gz-sim-ros2-control-system">
+        <robot_namespace>ur3e</robot_namespace>
+        <parameters>package://ur_custom_description/config/ur3e_controllers.yaml</parameters>
+      </plugin>
+    </gazebo>
     <!-- Include macros for the UR3e and the OnRobot 2FG7 gripper -->
-    <xacro:include filename="$(find ur_custom_description)/urdf/ur3e_urdf.xacro" />
-    <xacro:include filename="$(find ur_custom_description)/urdf/onrobot_2fg7_urdf.xacro" />
-    <xacro:include filename="$(find ur_custom_description)/urdf/realsense_L515_urdf.xacro" />
+    <xacro:include filename="ur3e_urdf.xacro" />
+    <xacro:include filename="onrobot_2fg7_urdf.xacro" />
+    <xacro:include filename="realsense_L515_urdf.xacro" />
 </robot>
