Commit message: RViz UR3e, 2FG7 and L515 (simple)

File: src/ur_custom/ur_custom_description/urdf/onrobot_2fg7_urdf.xacro (robot description, xacro)
@@ -53,5 +53,5 @@
       <origin rpy="0 0 0" xyz="0 0 0"/>
       <geometry>
-        <mesh filename="package://ur_robotiq_description/meshes/base_link.stl" scale="0.001 0.001 0.001"/>
+        <mesh filename="package://ur_custom_description/meshes/base_link.stl" scale="0.001 0.001 0.001"/>
       </geometry>
       <material name="silver"/>
@@ -60,5 +60,5 @@
       <origin rpy="0 0 0" xyz="0 0 0"/>
       <geometry>
-        <mesh filename="package://ur_robotiq_description/meshes/base_link.stl" scale="0.001 0.001 0.001"/>
+        <mesh filename="package://ur_custom_description/meshes/base_link.stl" scale="0.001 0.001 0.001"/>
       </geometry>
     </collision>
@@ -73,5 +73,5 @@
       <origin rpy="0 0 0" xyz="0.054361 0.029494 -0.12005"/>
       <geometry>
-        <mesh filename="package://ur_robotiq_description/meshes/right_finger_link.stl" scale="0.001 0.001 0.001"/>
+        <mesh filename="package://ur_custom_description/meshes/right_finger_link.stl" scale="0.001 0.001 0.001"/>
       </geometry>
       <material name="silver"/>
@@ -80,5 +80,5 @@
       <origin rpy="0 0 0" xyz="0.054361 0.029494 -0.12005"/>
       <geometry>
-        <mesh filename="package://ur_robotiq_description/meshes/right_finger_link.stl" scale="0.001 0.001 0.001"/>
+        <mesh filename="package://ur_custom_description/meshes/right_finger_link.stl" scale="0.001 0.001 0.001"/>
       </geometry>
     </collision>
@@ -93,5 +93,5 @@
       <origin rpy="0 0 0" xyz="-0.032239 0.029494 -0.12005"/>
       <geometry>
-        <mesh filename="package://ur_robotiq_description/meshes/left_finger_link.stl" scale="0.001 0.001 0.001"/>
+        <mesh filename="package://ur_custom_description/meshes/left_finger_link.stl" scale="0.001 0.001 0.001"/>
       </geometry>
       <material name="silver"/>
@@ -100,5 +100,5 @@
       <origin rpy="0 0 0" xyz="-0.032239 0.029494 -0.12005"/>
       <geometry>
-        <mesh filename="package://ur_robotiq_description/meshes/left_finger_link.stl" scale="0.001 0.001 0.001"/>
+        <mesh filename="package://ur_custom_description/meshes/left_finger_link.stl" scale="0.001 0.001 0.001"/>
       </geometry>
     </collision>

File: src/ur_custom/ur_custom_description/urdf/realsense_L515_urdf.xacro (robot description, xacro)
@@ -24,5 +24,5 @@
   </link>
   <joint name="gripper_to_l515" type="fixed">
-    <parent link="onrobot_2fg7_base_link"/>
+    <parent link="tool0"/>
     <child link="l515_base"/>
     <origin rpy="0 0 0" xyz="0 0 0"/>

File: src/ur_custom/ur_custom_description/urdf/ur3e_urdf.xacro (robot description, xacro)
@@ -1,7 +1,3 @@
 <?xml version="1.0" ?>
-<!-- =================================================================================== -->
-<!-- |    This document was autogenerated by xacro from ur3e.xacro                     | -->
-<!-- |    EDITING THIS FILE BY HAND IS NOT RECOMMENDED                                 | -->
-<!-- =================================================================================== -->
 <robot name="ur3e_robot">
   <!--

Commit message: Gazebo removed

File: src/ur_custom/ur_custom_description/urdf/onrobot_2fg7_urdf.xacro (robot description, xacro)
@@ -4,44 +4,4 @@
     <color rgba="0.700 0.700 0.700 1.000"/>
   </material>
-  <gazebo reference="onrobot_2fg7_base_link">
-    <material>Gazebo/Grey</material>
-    <implicitSpringDamper>1</implicitSpringDamper>
-    <mu1>0.2</mu1>
-    <mu2>0.2</mu2>
-    <kp>100000000.0</kp>
-    <kd>1.0</kd>
-    <selfCollide>true</selfCollide>
-    <gravity>true</gravity>
-  </gazebo>
-  <gazebo reference="right_finger_link">
-    <material>Gazebo/Grey</material>
-    <implicitSpringDamper>1</implicitSpringDamper>
-    <mu1>0.2</mu1>
-    <mu2>0.2</mu2>
-    <kp>100000000.0</kp>
-    <kd>1.0</kd>
-    <selfCollide>true</selfCollide>
-  </gazebo>
-  <gazebo reference="left_finger_link">
-    <material>Gazebo/Grey</material>
-    <implicitSpringDamper>1</implicitSpringDamper>
-    <mu1>0.2</mu1>
-    <mu2>0.2</mu2>
-    <kp>100000000.0</kp>
-    <kd>1.0</kd>
-    <selfCollide>true</selfCollide>
-  </gazebo>
-  <!--
-  <transmission name="left_finger_joint_tran">
-    <type>transmission_interface/SimpleTransmission</type>
-    <joint name="left_finger_joint">
-      <hardwareInterface>hardware_interface/PositionJointInterface</hardwareInterface>
-    </joint>
-    <actuator name="left_finger_joint_motor">
-      <hardwareInterface>hardware_interface/PositionJointInterface</hardwareInterface>
-      <mechanicalReduction>1</mechanicalReduction>
-    </actuator>
-  </transmission>
-  -->
   <link name="onrobot_2fg7_base_link">
     <inertial>
@@ -126,29 +86,3 @@
     <origin rpy="0.0 0.0 0.0" xyz="0.0 0.0 0.0"/>
   </joint>
-  <gazebo>
-    <plugin filename="libgazebo_grasp_fix.so" name="gazebo_grasp_fix">
-      <arm>
-        <arm_name>2FG7</arm_name>
-        <palm_link>onrobot_2fg7_base_link</palm_link>
-        <gripper_link>left_finger_link</gripper_link>
-        <gripper_link>right_finger_link</gripper_link>
-      </arm>
-      <forces_angle_tolerance>80</forces_angle_tolerance>
-      <update_rate>10</update_rate>
-      <grip_count_threshold>1</grip_count_threshold>
-      <max_grip_count>3</max_grip_count>
-      <release_tolerance>0.01</release_tolerance>
-      <disable_collisions_on_attach>false</disable_collisions_on_attach>
-      <contact_topic>__default_topic__</contact_topic>
-    </plugin>
-  </gazebo>
-  <!-- loading plugin: mimic joints works in gazebo now -->
-  <gazebo>
-    <plugin filename="libroboticsgroup_upatras_gazebo_mimic_joint_plugin.so" name="mimic_2FG7">
-      <joint>left_finger_joint</joint>
-      <mimicJoint>right_finger_joint</mimicJoint>
-      <multiplier>1.0</multiplier>
-      <offset>0.0</offset>
-    </plugin>
-  </gazebo>
 </robot>

File: src/ur_custom/ur_custom_description/urdf/realsense_L515_urdf.xacro (robot description, xacro)
@@ -1,27 +1,4 @@
 <?xml version="1.0" ?>
 <robot name="realsense_L515_camera">
-  <gazebo reference="l515_camera_link">
-    <sensor name="l515_camera" type="camera">
-      <camera>
-        <horizontal_fov>1.047</horizontal_fov> <!-- 60 degrees -->
-        <image>
-          <width>1280</width>
-          <height>720</height>
-          <format>R8G8B8</format>
-        </image>
-        <clip>
-          <near>0.1</near>
-          <far>100.0</far>
-        </clip>
-      </camera>
-      <plugin name="camera_controller" filename="gz-sim-camera-system">
-        <ros>
-          <namespace>/l515</namespace>
-          <remapping>image_raw:=image_raw</remapping>
-          <remapping>camera_info:=camera_info</remapping>
-        </ros>
-      </plugin>
-    </sensor>
-  </gazebo>
   <link name="l515_base">
     <visual>

File: src/ur_custom/ur_custom_description/urdf/ur3e_onrobot_2fg7_urdf.xacro (robot description, xacro)
@@ -3,11 +3,4 @@
 	<!-- This xacro file combines the UR3e collaborative robotic arm, the
 		OnRobot 2FG7 gripper and a simplified version of the Realsense L515 Camera. -->
-    <!-- Gazebo plugin for ROS 2 joint control-->
-	<gazebo>
-      <plugin name="gz_ros2_control" filename="gz-sim-ros2-control-system">
-        <robot_namespace>ur3e</robot_namespace>
-        <parameters>package://ur_custom_description/config/ur3e_controllers.yaml</parameters>
-      </plugin>
-    </gazebo>
     <!-- Include macros for the UR3e and the OnRobot 2FG7 gripper -->
     <xacro:include filename="ur3e_urdf.xacro" />
