Commit message: Setting Moveit 2

File: src/ur_custom/ur_custom_description/urdf/mech/onrobot_2fg7_urdf.xacro (robot description, xacro)
@@ -80,5 +80,4 @@
     <mimic joint="left_finger_joint" multiplier="1.0"/>
   </joint>
-  <!-- <link name="base_link"/> -->
   <joint name="world_joint" type="fixed">
     <parent link="tool0"/>

File: src/ur_custom/ur_custom_description/urdf/mech/ur3e_urdf.xacro (robot description, xacro)
@@ -15,58 +15,4 @@
     calibration from the controller and generate the required .yaml file.
   -->
-  <transmission name="shoulder_pan_trans">
-    <type>transmission_interface/SimpleTransmission</type>
-    <joint name="shoulder_pan_joint">
-      <hardwareInterface>hardware_interface/PositionJointInterface</hardwareInterface>
-    </joint>
-    <actuator name="shoulder_pan_motor">
-      <mechanicalReduction>1</mechanicalReduction>
-    </actuator>
-  </transmission>
-  <transmission name="shoulder_lift_trans">
-    <type>transmission_interface/SimpleTransmission</type>
-    <joint name="shoulder_lift_joint">
-      <hardwareInterface>hardware_interface/PositionJointInterface</hardwareInterface>
-    </joint>
-    <actuator name="shoulder_lift_motor">
-      <mechanicalReduction>1</mechanicalReduction>
-    </actuator>
-  </transmission>
-  <transmission name="elbow_trans">
-    <type>transmission_interface/SimpleTransmission</type>
-    <joint name="elbow_joint">
-      <hardwareInterface>hardware_interface/PositionJointInterface</hardwareInterface>
-    </joint>
-    <actuator name="elbow_motor">
-      <mechanicalReduction>1</mechanicalReduction>
-    </actuator>
-  </transmission>
-  <transmission name="wrist_1_trans">
-    <type>transmission_interface/SimpleTransmission</type>
-    <joint name="wrist_1_joint">
-      <hardwareInterface>hardware_interface/PositionJointInterface</hardwareInterface>
-    </joint>
-    <actuator name="wrist_1_motor">
-      <mechanicalReduction>1</mechanicalReduction>
-    </actuator>
-  </transmission>
-  <transmission name="wrist_2_trans">
-    <type>transmission_interface/SimpleTransmission</type>
-    <joint name="wrist_2_joint">
-      <hardwareInterface>hardware_interface/PositionJointInterface</hardwareInterface>
-    </joint>
-    <actuator name="wrist_2_motor">
-      <mechanicalReduction>1</mechanicalReduction>
-    </actuator>
-  </transmission>
-  <transmission name="wrist_3_trans">
-    <type>transmission_interface/SimpleTransmission</type>
-    <joint name="wrist_3_joint">
-      <hardwareInterface>hardware_interface/PositionJointInterface</hardwareInterface>
-    </joint>
-    <actuator name="wrist_3_motor">
-      <mechanicalReduction>1</mechanicalReduction>
-    </actuator>
-  </transmission>
   <!-- links: main serial chain -->
   <link name="base_link"/>
@@ -285,7 +231,7 @@
     <dynamics damping="0" friction="0"/>
   </joint>
-  <!-- ROS-Industrial 'base' frame: base_link to UR 'Base' Coordinates transform -->
-  <link name="base"/>
-  <joint name="base_link-base_fixed_joint" type="fixed">
+  <!-- ROS-Industrial 'base' frame: base_link to UR 'world' Coordinates transform -->
+  <link name="world"/>
+  <joint name="base_link-world" type="fixed">
     <!-- Note the rotation over Z of pi radians: as base_link is REP-103
            aligned (ie: has X+ forward, Y+ left and Z+ up), this is needed
@@ -295,5 +241,5 @@
     <origin rpy="0 0 3.141592653589793" xyz="0 0 0"/>
     <parent link="base_link"/>
-    <child link="base"/>
+    <child link="world"/>
   </joint>
   <!-- ROS-Industrial 'flange' frame: attachment point for EEF models -->

File: src/ur_custom/ur_custom_description/urdf/robots/ur3e_onrobot_2fg7_urdf.xacro (robot description, xacro)
@@ -4,6 +4,6 @@
 		OnRobot 2FG7 gripper and a simplified version of the Realsense L515 Camera. -->
     <!-- Include macros for the UR3e and the OnRobot 2FG7 gripper -->
-    <xacro:include filename="ur3e_urdf.xacro" />
-    <xacro:include filename="onrobot_2fg7_urdf.xacro" />
-    <xacro:include filename="realsense_L515_urdf.xacro" />
+    <xacro:include filename="../mech/ur3e_urdf.xacro" />
+    <xacro:include filename="../mech/onrobot_2fg7_urdf.xacro" />
+    <xacro:include filename="../sensors/realsense_L515_urdf.xacro" />
 </robot>

Commit message: Setting Moveit 2

File: src/ur_custom/ur_custom_description/urdf/mech/onrobot_2fg7_urdf.xacro (robot description, xacro)
@@ -13,5 +13,5 @@
       <origin rpy="0 0 0" xyz="0 0 0"/>
       <geometry>
-        <mesh filename="package://ur_custom_description/meshes/base_link.stl" scale="0.001 0.001 0.001"/>
+        <mesh filename="package://ur_custom_description/meshes/onrobot_2fg7/base_link.stl" scale="0.001 0.001 0.001"/>
       </geometry>
       <material name="silver"/>
@@ -20,5 +20,5 @@
       <origin rpy="0 0 0" xyz="0 0 0"/>
       <geometry>
-        <mesh filename="package://ur_custom_description/meshes/base_link.stl" scale="0.001 0.001 0.001"/>
+        <mesh filename="package://ur_custom_description/meshes/onrobot_2fg7/base_link.stl" scale="0.001 0.001 0.001"/>
       </geometry>
     </collision>
@@ -33,5 +33,5 @@
       <origin rpy="0 0 0" xyz="0.054361 0.029494 -0.12005"/>
       <geometry>
-        <mesh filename="package://ur_custom_description/meshes/right_finger_link.stl" scale="0.001 0.001 0.001"/>
+        <mesh filename="package://ur_custom_description/meshes/onrobot_2fg7/right_finger_link.stl" scale="0.001 0.001 0.001"/>
       </geometry>
       <material name="silver"/>
@@ -40,5 +40,5 @@
       <origin rpy="0 0 0" xyz="0.054361 0.029494 -0.12005"/>
       <geometry>
-        <mesh filename="package://ur_custom_description/meshes/right_finger_link.stl" scale="0.001 0.001 0.001"/>
+        <mesh filename="package://ur_custom_description/meshes/onrobot_2fg7/right_finger_link.stl" scale="0.001 0.001 0.001"/>
       </geometry>
     </collision>
@@ -53,5 +53,5 @@
       <origin rpy="0 0 0" xyz="-0.032239 0.029494 -0.12005"/>
       <geometry>
-        <mesh filename="package://ur_custom_description/meshes/left_finger_link.stl" scale="0.001 0.001 0.001"/>
+        <mesh filename="package://ur_custom_description/meshes/onrobot_2fg7/left_finger_link.stl" scale="0.001 0.001 0.001"/>
       </geometry>
       <material name="silver"/>
@@ -60,5 +60,5 @@
       <origin rpy="0 0 0" xyz="-0.032239 0.029494 -0.12005"/>
       <geometry>
-        <mesh filename="package://ur_custom_description/meshes/left_finger_link.stl" scale="0.001 0.001 0.001"/>
+        <mesh filename="package://ur_custom_description/meshes/onrobot_2fg7/left_finger_link.stl" scale="0.001 0.001 0.001"/>
       </geometry>
     </collision>

File: src/ur_custom/ur_custom_description/urdf/sensors/realsense_L515_urdf.xacro (robot description, xacro)
@@ -4,6 +4,11 @@
     <visual>
       <origin rpy="0 0 0" xyz="0 -0.07 -0.01"/>
+      <!--
       <geometry>
         <cylinder radius="0.03" length="0.04"/>
+      </geometry>
+      -->
+      <geometry>
+        <mesh filename="package://ur_custom_description/meshes/realsense_l515/Intel_RealSense_L515.stl" scale="1 1 1"/>
       </geometry>
       <material name="black">
