Commit message: Setting Moveit 2

File: src/ur_custom/ur_custom_description/urdf/mech/robotiq_2f_85_urdf.xacro (robot description, xacro)
@@ -31,10 +31,10 @@
             <visual>
                 <geometry>
-                    <mesh filename="file://$(find robotiq_description)/meshes/visual/robotiq_base.dae" />
-                </geometry>
-            </visual>
-            <collision>
-                <geometry>
-                    <mesh filename="file://$(find robotiq_description)/meshes/collision/robotiq_base.stl" />
+                    <mesh filename="package://ur_custom_description/meshes/robotiq_2f_85/visual/robotiq_base.dae" />
+                </geometry>
+            </visual>
+            <collision>
+                <geometry>
+                    <mesh filename="package://ur_custom_description/meshes/robotiq_2f_85/collision/robotiq_base.stl" />
                 </geometry>
             </collision>
@@ -48,10 +48,10 @@
             <visual>
                 <geometry>
-                    <mesh filename="file://$(find robotiq_description)/meshes/visual/left_knuckle.dae" />
-                </geometry>
-            </visual>
-            <collision>
-                <geometry>
-                    <mesh filename="file://$(find robotiq_description)/meshes/collision/left_knuckle.stl" />
+                    <mesh filename="package://ur_custom_description/meshes/robotiq_2f_85/visual/left_knuckle.dae" />
+                </geometry>
+            </visual>
+            <collision>
+                <geometry>
+                    <mesh filename="package://ur_custom_description/meshes/robotiq_2f_85/collision/left_knuckle.stl" />
                 </geometry>
             </collision>
@@ -65,10 +65,10 @@
             <visual>
                 <geometry>
-                    <mesh filename="file://$(find robotiq_description)/meshes/visual/right_knuckle.dae" />
-                </geometry>
-            </visual>
-            <collision>
-                <geometry>
-                    <mesh filename="file://$(find robotiq_description)/meshes/collision/right_knuckle.stl" />
+                    <mesh filename="package://ur_custom_description/meshes/robotiq_2f_85/visual/right_knuckle.dae" />
+                </geometry>
+            </visual>
+            <collision>
+                <geometry>
+                    <mesh filename="package://ur_custom_description/meshes/robotiq_2f_85/collision/right_knuckle.stl" />
                 </geometry>
             </collision>
@@ -82,10 +82,10 @@
             <visual>
                 <geometry>
-                    <mesh filename="file://$(find robotiq_description)/meshes/visual/left_finger.dae" />
-                </geometry>
-            </visual>
-            <collision>
-                <geometry>
-                    <mesh filename="file://$(find robotiq_description)/meshes/collision/left_finger.stl" />
+                    <mesh filename="package://ur_custom_description/meshes/robotiq_2f_85/visual/left_finger.dae" />
+                </geometry>
+            </visual>
+            <collision>
+                <geometry>
+                    <mesh filename="package://ur_custom_description/meshes/robotiq_2f_85/collision/left_finger.stl" />
                 </geometry>
             </collision>
@@ -99,10 +99,10 @@
             <visual>
                 <geometry>
-                    <mesh filename="file://$(find robotiq_description)/meshes/visual/right_finger.dae" />
-                </geometry>
-            </visual>
-            <collision>
-                <geometry>
-                    <mesh filename="file://$(find robotiq_description)/meshes/collision/right_finger.stl" />
+                    <mesh filename="package://ur_custom_description/meshes/robotiq_2f_85/visual/right_finger.dae" />
+                </geometry>
+            </visual>
+            <collision>
+                <geometry>
+                    <mesh filename="package://ur_custom_description/meshes/robotiq_2f_85/collision/right_finger.stl" />
                 </geometry>
             </collision>
@@ -116,10 +116,10 @@
             <visual>
                 <geometry>
-                    <mesh filename="file://$(find robotiq_description)/meshes/visual/left_inner_knuckle.dae" />
-                </geometry>
-            </visual>
-            <collision>
-                <geometry>
-                    <mesh filename="file://$(find robotiq_description)/meshes/collision/left_inner_knuckle.stl" />
+                    <mesh filename="package://ur_custom_description/meshes/robotiq_2f_85/visual/left_inner_knuckle.dae" />
+                </geometry>
+            </visual>
+            <collision>
+                <geometry>
+                    <mesh filename="package://ur_custom_description/meshes/robotiq_2f_85/collision/left_inner_knuckle.stl" />
                 </geometry>
             </collision>
@@ -133,10 +133,10 @@
             <visual>
                 <geometry>
-                    <mesh filename="file://$(find robotiq_description)/meshes/visual/right_inner_knuckle.dae" />
-                </geometry>
-            </visual>
-            <collision>
-                <geometry>
-                    <mesh filename="file://$(find robotiq_description)/meshes/collision/right_inner_knuckle.stl" />
+                    <mesh filename="package://ur_custom_description/meshes/robotiq_2f_85/visual/right_inner_knuckle.dae" />
+                </geometry>
+            </visual>
+            <collision>
+                <geometry>
+                    <mesh filename="package://ur_custom_description/meshes/robotiq_2f_85/collision/right_inner_knuckle.stl" />
                 </geometry>
             </collision>
@@ -150,10 +150,10 @@
             <visual>
                 <geometry>
-                    <mesh filename="file://$(find robotiq_description)/meshes/visual/left_finger_tip.dae" />
-                </geometry>
-            </visual>
-            <collision>
-                <geometry>
-                    <mesh filename="file://$(find robotiq_description)/meshes/collision/left_finger_tip.stl" />
+                    <mesh filename="package://ur_custom_description/meshes/robotiq_2f_85/visual/left_finger_tip.dae" />
+                </geometry>
+            </visual>
+            <collision>
+                <geometry>
+                    <mesh filename="package://ur_custom_description/meshes/robotiq_2f_85/collision/left_finger_tip.stl" />
                 </geometry>
                 <surface>
@@ -185,10 +185,10 @@
             <visual>
                 <geometry>
-                    <mesh filename="file://$(find robotiq_description)/meshes/visual/right_finger_tip.dae" />
-                </geometry>
-            </visual>
-            <collision>
-                <geometry>
-                    <mesh filename="file://$(find robotiq_description)/meshes/collision/right_finger_tip.stl" />
+                    <mesh filename="package://ur_custom_description/meshes/robotiq_2f_85/visual/right_finger_tip.dae" />
+                </geometry>
+            </visual>
+            <collision>
+                <geometry>
+                    <mesh filename="package://ur_custom_description/meshes/robotiq_2f_85/collision/right_finger_tip.stl" />
                 </geometry>
                 <surface>

File: src/ur_custom/ur_custom_description/urdf/mech/ur3e_urdf.xacro (robot description, xacro)
@@ -21,14 +21,14 @@
       <origin rpy="0 0 3.141592653589793" xyz="0 0 0"/>
       <geometry>
-        <mesh filename="package://ur_description/meshes/ur3e/visual/base.dae"/>
-      </geometry>
-      <material name="LightGrey">
-        <color rgba="0.7 0.7 0.7 1.0"/>
-      </material>
-    </visual>
-    <collision>
-      <origin rpy="0 0 3.141592653589793" xyz="0 0 0"/>
-      <geometry>
-        <mesh filename="package://ur_description/meshes/ur3e/collision/base.stl"/>
+        <mesh filename="package://ur_custom_description/meshes/ur3e/visual/base.dae"/>
+      </geometry>
+      <material name="LightGrey">
+        <color rgba="0.7 0.7 0.7 1.0"/>
+      </material>
+    </visual>
+    <collision>
+      <origin rpy="0 0 3.141592653589793" xyz="0 0 0"/>
+      <geometry>
+        <mesh filename="package://ur_custom_description/meshes/ur3e/collision/base.stl"/>
       </geometry>
     </collision>
@@ -43,14 +43,14 @@
       <origin rpy="0 0 3.141592653589793" xyz="0 0 0"/>
       <geometry>
-        <mesh filename="package://ur_description/meshes/ur3e/visual/shoulder.dae"/>
-      </geometry>
-      <material name="LightGrey">
-        <color rgba="0.7 0.7 0.7 1.0"/>
-      </material>
-    </visual>
-    <collision>
-      <origin rpy="0 0 3.141592653589793" xyz="0 0 0"/>
-      <geometry>
-        <mesh filename="package://ur_description/meshes/ur3e/collision/shoulder.stl"/>
+        <mesh filename="package://ur_custom_description/meshes/ur3e/visual/shoulder.dae"/>
+      </geometry>
+      <material name="LightGrey">
+        <color rgba="0.7 0.7 0.7 1.0"/>
+      </material>
+    </visual>
+    <collision>
+      <origin rpy="0 0 3.141592653589793" xyz="0 0 0"/>
+      <geometry>
+        <mesh filename="package://ur_custom_description/meshes/ur3e/collision/shoulder.stl"/>
       </geometry>
     </collision>
@@ -65,5 +65,5 @@
       <origin rpy="1.5707963267948966 0 -1.5707963267948966" xyz="0 0 0.12"/>
       <geometry>
-        <mesh filename="package://ur_description/meshes/ur3e/visual/upperarm.dae"/>
+        <mesh filename="package://ur_custom_description/meshes/ur3e/visual/upperarm.dae"/>
       </geometry>
       <material name="LightGrey">
@@ -74,5 +74,5 @@
       <origin rpy="1.5707963267948966 0 -1.5707963267948966" xyz="0 0 0.12"/>
       <geometry>
-        <mesh filename="package://ur_description/meshes/ur3e/collision/upperarm.stl"/>
+        <mesh filename="package://ur_custom_description/meshes/ur3e/collision/upperarm.stl"/>
       </geometry>
     </collision>
@@ -87,5 +87,5 @@
       <origin rpy="1.5707963267948966 0 -1.5707963267948966" xyz="0 0 0.027"/>
       <geometry>
-        <mesh filename="package://ur_description/meshes/ur3e/visual/forearm.dae"/>
+        <mesh filename="package://ur_custom_description/meshes/ur3e/visual/forearm.dae"/>
       </geometry>
       <material name="LightGrey">
@@ -96,5 +96,5 @@
       <origin rpy="1.5707963267948966 0 -1.5707963267948966" xyz="0 0 0.027"/>
       <geometry>
-        <mesh filename="package://ur_description/meshes/ur3e/collision/forearm.stl"/>
+        <mesh filename="package://ur_custom_description/meshes/ur3e/collision/forearm.stl"/>
       </geometry>
     </collision>
@@ -110,5 +110,5 @@
       <origin rpy="1.5707963267948966 0 0" xyz="0 0 -0.104"/>
       <geometry>
-        <mesh filename="package://ur_description/meshes/ur3e/visual/wrist1.dae"/>
+        <mesh filename="package://ur_custom_description/meshes/ur3e/visual/wrist1.dae"/>
       </geometry>
       <material name="LightGrey">
@@ -119,5 +119,5 @@
       <origin rpy="1.5707963267948966 0 0" xyz="0 0 -0.104"/>
       <geometry>
-        <mesh filename="package://ur_description/meshes/ur3e/collision/wrist1.stl"/>
+        <mesh filename="package://ur_custom_description/meshes/ur3e/collision/wrist1.stl"/>
       </geometry>
     </collision>
@@ -132,5 +132,5 @@
       <origin rpy="0 0 0" xyz="0 0 -0.08535"/>
       <geometry>
-        <mesh filename="package://ur_description/meshes/ur3e/visual/wrist2.dae"/>
+        <mesh filename="package://ur_custom_description/meshes/ur3e/visual/wrist2.dae"/>
       </geometry>
       <material name="LightGrey">
@@ -141,5 +141,5 @@
       <origin rpy="0 0 0" xyz="0 0 -0.08535"/>
       <geometry>
-        <mesh filename="package://ur_description/meshes/ur3e/collision/wrist2.stl"/>
+        <mesh filename="package://ur_custom_description/meshes/ur3e/collision/wrist2.stl"/>
       </geometry>
     </collision>
@@ -154,5 +154,5 @@
       <origin rpy="1.5707963267948966 0 0" xyz="0 0 -0.0921"/>
       <geometry>
-        <mesh filename="package://ur_description/meshes/ur3e/visual/wrist3.dae"/>
+        <mesh filename="package://ur_custom_description/meshes/ur3e/visual/wrist3.dae"/>
       </geometry>
       <material name="LightGrey">
@@ -163,5 +163,5 @@
       <origin rpy="1.5707963267948966 0 0" xyz="0 0 -0.0921"/>
       <geometry>
-        <mesh filename="package://ur_description/meshes/ur3e/collision/wrist3.stl"/>
+        <mesh filename="package://ur_custom_description/meshes/ur3e/collision/wrist3.stl"/>
       </geometry>
     </collision>

File: src/ur_custom/ur_custom_description/urdf/sensors/realsense_L515_urdf.xacro (robot description, xacro)
@@ -1,35 +1,97 @@
 <?xml version="1.0" ?>
-<robot name="realsense_L515_camera">
-  <link name="l515_base">
-    <visual>
-      <origin rpy="0 0 0" xyz="0 -0.07 -0.01"/>
-      <!--
-      <geometry>
-        <cylinder radius="0.03" length="0.04"/>
-      </geometry>
-      -->
-      <geometry>
-        <mesh filename="package://ur_custom_description/meshes/realsense_l515/Intel_RealSense_L515.stl" scale="1 1 1"/>
-      </geometry>
-      <material name="black">
-        <color rgba="0.0 0.0 0.0 1.0"/>
-      </material>
-    </visual>
-    <collision>
-      <origin rpy="0 0 0" xyz="0 -0.07 -0.01"/>
-      <geometry>
-        <cylinder radius="0.03" length="0.04"/>
-      </geometry>
-    </collision>
-    <inertial>
-      <origin rpy="0 0 0" xyz="0 -0.07 -0.01"/>
-      <mass value="0.1"/>
-      <inertia ixx="0.0001" ixy="0.0" ixz="0.0" iyy="0.0001" iyz="0.0" izz="0.0001"/>
-    </inertial>
-  </link>
-  <joint name="gripper_to_l515" type="fixed">
-    <parent link="tool0"/>
-    <child link="l515_base"/>
-    <origin rpy="0 0 0" xyz="0 0 0"/>
-  </joint>
+<robot xmlns:xacro="http://www.ros.org/wiki/xacro">
+  <xacro:arg name="use_camera" default="true"/>
+  <xacro:arg name="use_gazebo" default="true"/>
+  <xacro:arg name="prefix" default=""/>
+  <xacro:if value="${'true' == '$(arg use_camera)' and 'true' == '$(arg use_gazebo)'}">
+  <xacro:property name="M_PI" value="3.1415926535897931" />
+  <xacro:property name="l515_cam_width" value="0.061"/>
+  <xacro:property name="l515_cam_height" value="0.061"/>
+  <xacro:property name="l515_cam_depth" value="0.026"/>
+  <xacro:property name="l515_cam_depth_to_infra_offset" value="0.0"/>
+  <xacro:property name="l515_cam_depth_to_color_offset" value="0.012"/>
+    <joint name="camera_joint" type="fixed">
+      <parent link="tool0"/>
+      <child link="camera" />
+      <origin xyz="0 0 0" rpy="0 0 0"/>
+    </joint>
+    <link name="camera">
+      <visual>
+        <origin rpy="0 0 0" xyz="0 -0.07 -0.01"/>
+        <geometry>
+          <mesh filename="package://ur_custom_description/meshes/realsense_l515/Intel_RealSense_L515.stl" scale="0.001 0.001 0.001"/>
+        </geometry>
+        <material name="aluminum">
+          <color rgba="0.5 0.5 0.5 1"/>
+        </material>
+      </visual>
+      <collision>
+        <origin rpy="0 0 0" xyz="0 -0.07 -0.01"/>
+        <geometry>
+          <box size="${l515_cam_depth} ${l515_cam_width} ${l515_cam_height}"/>
+        </geometry>
+      </collision>
+      <inertial>
+        <mass value="0.095" />
+        <origin rpy="0 0 0" xyz="0 -0.07 -0.01"/>
+        <inertia ixx="0.000044" ixy="0.0" ixz="0.0" iyy="0.000027" iyz="0.0" izz="0.000027" />
+      </inertial>
+    </link>
+    <joint name="camera_depth_joint" type="fixed">
+      <origin xyz="0 0 0" rpy="0 0 0"/>
+      <parent link="camera"/>
+      <child link="camera_depth_frame" />
+    </joint>
+    <link name="camera_depth_frame"/>
+    <joint name="camera_depth_optical_joint" type="fixed">
+      <origin xyz="0 0 0" rpy="0 0 0" />
+      <parent link="camera_depth_frame" />
+      <child link="camera_depth_optical_frame" />
+    </joint>
+    <link name="camera_depth_optical_frame"/>
+    <joint name="camera_infra_joint" type="fixed">
+      <origin xyz="0 ${l515_cam_depth_to_infra_offset} 0" rpy="0 0 0" />
+      <parent link="camera" />
+      <child link="camera_infra_frame" />
+    </joint>
+    <link name="camera_infra_frame"/>
+    <joint name="camera_infra_optical_joint" type="fixed">
+      <origin xyz="0 0 0" rpy="0 0 0" />
+      <parent link="camera_infra_frame" />
+      <child link="camera_infra_optical_frame" />
+    </joint>
+    <link name="camera_infra_optical_frame"/>
+    <joint name="camera_color_joint" type="fixed">
+      <origin xyz="0 ${l515_cam_depth_to_color_offset} 0" rpy="0 0 0" />
+      <parent link="camera" />
+      <child link="camera_color_frame" />
+    </joint>
+    <link name="camera_color_frame"/>
+    <joint name="camera_color_optical_joint" type="fixed">
+      <origin xyz="0 0 0" rpy="0 0 0" />
+      <parent link="camera_color_frame" />
+      <child link="camera_color_optical_frame" />
+    </joint>
+    <link name="camera_color_optical_frame"/>
+    <gazebo reference="camera">
+      <sensor name="camera_rgbd" type="rgbd_camera">
+        <camera>
+          <horizontal_fov>1.5184</horizontal_fov>
+          <image>
+            <width>1920</width>
+            <height>1080</height>
+          </image>
+          <clip>
+            <near>0.25</near>
+            <far>9</far>
+          </clip>
+        </camera>
+        <always_on>1</always_on>
+        <gz_frame_id>camera_head_link</gz_frame_id>
+        <topic>camera_head</topic>
+        <update_rate>5</update_rate>
+        <visualize>true</visualize>
+      </sensor>
+    </gazebo>
+  </xacro:if>
 </robot>
