Commit message: Moveit 2, Gazebo and ROS 2 control

File: src/ur_custom/ur_custom_description/urdf/mech/adaptive_gripper.urdf.xacro (robot description, xacro)
@@ -10,4 +10,7 @@
   <xacro:property name="gripper_link_izz" value="2e-06"/>
   <xacro:macro name="adaptive_gripper" params="parent prefix *origin">
+    <material name="silver">
+      <color rgba="0.600 0.600 0.600 1.000"/>
+    </material>
     <link name="${prefix}gripper_base">
       <inertial>
@@ -21,7 +24,8 @@
       <visual>
         <geometry>
-          <mesh filename="file://$(find ur_custom_description)/meshes/onrobot_2fg7/visual/base_link.stl" scale="0.001 0.001 0.001"/>
+          <mesh filename="file://$(find ur_custom_description)/meshes/onrobot_2fg7/base_link.stl" scale="0.001 0.001 0.001"/>
         </geometry>
         <origin xyz="0 0 0" rpy="0 0 0"/>
+        <material name="silver"/>
       </visual>
       <collision>
@@ -48,11 +52,12 @@
       <visual>
         <geometry>
-          <mesh filename="file://$(find ur_custom_description)/meshes/onrobot_2fg7/left_finger_link.stl"/>
+          <mesh filename="file://$(find ur_custom_description)/meshes/onrobot_2fg7/left_finger_link.stl" scale="0.001 0.001 0.001"/>
         </geometry>
         <origin xyz="-0.032239 0.029494 -0.12005" rpy="0 0 0"/>
+        <material name="silver"/>
       </visual>
       <collision>
         <geometry>
-          <mesh filename="file://$(find ur_custom_description)/meshes/onrobot_2fg7/left_finger_link.stl"/>
+          <mesh filename="file://$(find ur_custom_description)/meshes/onrobot_2fg7/left_finger_link.stl" scale="0.001 0.001 0.001"/>
         </geometry>
         <origin xyz="-0.032239 0.029494 -0.12005" rpy="0 0 0"/>
@@ -70,11 +75,12 @@
       <visual>
         <geometry>
-          <mesh filename="file://$(find ur_custom_description)/meshes/onrobot_2fg7/right_finger_link.stl"/>
+          <mesh filename="file://$(find ur_custom_description)/meshes/onrobot_2fg7/right_finger_link.stl" scale="0.001 0.001 0.001"/>
         </geometry>
         <origin xyz="0.054361 0.029494 -0.12005" rpy="0 0 0"/>
+        <material name="silver"/>
       </visual>
       <collision>
         <geometry>
-          <mesh filename="file://$(find ur_custom_description)/meshes/onrobot_2fg7/right_finger_link.stl"/>
+          <mesh filename="file://$(find ur_custom_description)/meshes/onrobot_2fg7/right_finger_link.stl" scale="0.001 0.001 0.001"/>
         </geometry>
         <origin xyz="0.054361 0.029494 -0.12005" rpy="0 0 0"/>

File: src/ur_custom/ur_custom_description/urdf/mech/g_shape_base_v2_0.urdf.xacro (robot description, xacro)
@@ -13,5 +13,5 @@
             <visual>
                 <geometry>
-                    <mesh filename="file://$(find mycobot_description)/meshes/g_shape_base_v2_0/visual/base_link.dae"/>
+                    <mesh filename="file://$(find ur_custom_description)/meshes/g_shape_base_v2_0/visual/base_link.dae"/>
                 </geometry>
                 <origin xyz="0.0 0 -0.03" rpy="0 0 ${pi/2}"/>

File: src/ur_custom/ur_custom_description/urdf/mech/ur3e_arm.urdf.xacro (robot description, xacro)
@@ -156,7 +156,7 @@
       <axis xyz="0 0 1"/>
       <limit effort="${joint_effort}" lower="-6.283185307179586" upper="6.283185307179586" velocity="${joint_velocity}"/>
-      <parent link="${prefix}link3"/>
-      <child link="${prefix}link4"/>
-      <origin xyz="0 0 0" rpy="1.570796327 0 0/>
+      <parent link="${prefix}link2"/>
+      <child link="${prefix}link3"/>
+      <origin xyz="0 0 0" rpy="1.570796327 0 0"/>
       <dynamics damping="${joint_damping}" friction="${joint_friction}"/>
     </joint>
@@ -166,5 +166,5 @@
       <parent link="${prefix}link3"/>
       <child link="${prefix}link4"/>
-      <origin xyz="-0.24355 0 0" rpy="0 0 0/>
+      <origin xyz="-0.24355 0 0" rpy="0 0 0"/>
       <dynamics damping="${joint_damping}" friction="${joint_friction}"/>
     </joint>

File: src/ur_custom/ur_custom_description/urdf/robots/ur3e_2fg7_l515.urdf.xacro (robot description, xacro)
@@ -53,4 +53,4 @@
       flange_link="$(arg flange_link)"
       use_gazebo="$(arg use_gazebo)"/>
-    <xacro:include filename="$(find ur_custom_description)/urdf/sensors/intel_rgbd_cam_d435.urdf.xacro"/>
+    <xacro:include filename="$(find ur_custom_description)/urdf/sensors/intel_rgbd_cam_l515.urdf.xacro"/>
 </robot>

File: src/ur_custom/ur_custom_description/urdf/sensors/intel_rgbd_cam_l515.urdf.xacro (robot description, xacro)
@@ -4,4 +4,5 @@
   <xacro:arg name="use_gazebo" default="true"/>
   <xacro:arg name="prefix" default=""/>
+  <xacro:arg name="flange_link" default="link6_flange"/>
   <xacro:if value="${'true' == '$(arg use_camera)' and 'true' == '$(arg use_gazebo)'}">
   <xacro:property name="M_PI" value="3.1415926535897931" />
@@ -12,5 +13,5 @@
   <xacro:property name="l515_cam_depth_to_color_offset" value="0.012"/>
     <joint name="camera_joint" type="fixed">
-      <parent link="tool0"/>
+      <parent link="$(arg prefix)$(arg flange_link)"/>
       <child link="camera" />
       <origin xyz="0 0 0" rpy="0 0 0"/>
@@ -29,5 +30,5 @@
         <origin rpy="0 0 0" xyz="0 -0.07 -0.01"/>
         <geometry>
-          <box size="${l515_cam_depth} ${l515_cam_width} ${l515_cam_height}"/>
+          <mesh filename="package://ur_custom_description/meshes/realsense_l515/Intel_RealSense_L515.stl" scale="0.001 0.001 0.001"/>
         </geometry>
       </collision>
@@ -88,6 +89,6 @@
         </camera>
         <always_on>1</always_on>
-        <gz_frame_id>camera_head_link</gz_frame_id>
-        <topic>camera_head</topic>
+        <gz_frame_id>camera</gz_frame_id>
+        <topic>camera</topic>
         <update_rate>5</update_rate>
         <visualize>true</visualize>

Commit message: Fixing bugs for Gazebo

File: src/ur_custom/ur_custom_description/urdf/mech/adaptive_gripper.urdf.xacro (robot description, xacro)
@@ -1,5 +1,5 @@
 <?xml version="1.0"?>
 <robot xmlns:xacro="http://www.ros.org/wiki/xacro">
-  <xacro:property name="joint_effort" value="140"/>
+  <xacro:property name="joint_effort" value="140.0"/>
   <xacro:property name="joint_velocity" value="0.45"/>
   <xacro:property name="joint_damping" value="0.0"/>
