Commit message: Fix git

File: src/ur_custom/ur_custom_description/urdf/mech/gripper.urdf.xacro (robot description, xacro)
@@ -31,5 +31,5 @@
       <collision>
         <geometry>
-          <mesh filename="file://$(find ur_custom_description)/meshes/onrobot_2fg7/base_link.stl" scale="0.0012 0.0012 0.0012"/>
+          <mesh filename="file://$(find ur_custom_description)/meshes/onrobot_2fg7/base_link.stl" scale="0.0012 0.0012 0.001"/>
         </geometry>
         <origin xyz="0 0 0" rpy="0 0 0"/>
@@ -59,5 +59,5 @@
       <collision>
         <geometry>
-          <mesh filename="file://$(find ur_custom_description)/meshes/onrobot_2fg7/left_finger_link.stl" scale="0.0012 0.0012 0.0012"/>
+          <mesh filename="file://$(find ur_custom_description)/meshes/onrobot_2fg7/left_finger_link.stl" scale="0.0013 0.0013 0.001"/>
         </geometry>
         <origin xyz="-0.032239 0.029494 -0.12005" rpy="0 0 0"/>
@@ -82,5 +82,5 @@
       <collision>
         <geometry>
-          <mesh filename="file://$(find ur_custom_description)/meshes/onrobot_2fg7/right_finger_link.stl" scale="0.0012 0.0012 0.0012"/>
+          <mesh filename="file://$(find ur_custom_description)/meshes/onrobot_2fg7/right_finger_link.stl" scale="0.0013 0.0013 0.001"/>
         </geometry>
         <origin xyz="0.054361 0.029494 -0.12005" rpy="0 0 0"/>
