Commit message: Moveit 2, Gazebo and ROS 2 control

File: src/ur_custom/ur_custom_description/urdf/sensors/intel_rgbd_cam_l515.urdf.xacro (robot description, xacro)
@@ -6,20 +6,20 @@
   <xacro:arg name="flange_link" default="link6_flange"/>
   <xacro:if value="${'true' == '$(arg use_camera)' and 'true' == '$(arg use_gazebo)'}">
-  <xacro:property name="M_PI" value="3.1415926535897931" />
-  <xacro:property name="l515_cam_width" value="0.061"/>
-  <xacro:property name="l515_cam_height" value="0.061"/>
-  <xacro:property name="l515_cam_depth" value="0.026"/>
-  <xacro:property name="l515_cam_depth_to_infra_offset" value="0.0"/>
-  <xacro:property name="l515_cam_depth_to_color_offset" value="0.012"/>
+     <xacro:property name="M_PI" value="3.1415926535897931" />
+     <xacro:property name="l515_cam_width" value="0.061"/>
+     <xacro:property name="l515_cam_height" value="0.061"/>
+     <xacro:property name="l515_cam_depth" value="0.026"/>
+     <xacro:property name="l515_cam_depth_to_infra_offset" value="0.0"/>
+     <xacro:property name="l515_cam_depth_to_color_offset" value="0.012"/>
     <joint name="camera_joint" type="fixed">
       <parent link="$(arg prefix)$(arg flange_link)"/>
-      <child link="camera" />
+      <child link="camera_link" />
       <origin xyz="0 0 0" rpy="0 0 0"/>
     </joint>
-    <link name="camera">
+    <link name="camera_link">
       <visual>
         <origin rpy="0 0 0" xyz="0 -0.07 -0.01"/>
         <geometry>
-          <mesh filename="package://ur_custom_description/meshes/realsense_l515/Intel_RealSense_L515.stl" scale="0.001 0.001 0.001"/>
+          <mesh filename="file://$(find ur_custom_description)/meshes/realsense_l515/Intel_RealSense_L515.stl" scale="0.001 0.001 0.001"/>
         </geometry>
         <material name="aluminum">
@@ -30,5 +30,5 @@
         <origin rpy="0 0 0" xyz="0 -0.07 -0.01"/>
         <geometry>
-          <mesh filename="package://ur_custom_description/meshes/realsense_l515/Intel_RealSense_L515.stl" scale="0.001 0.001 0.001"/>
+          <mesh filename="file://$(find ur_custom_description)/meshes/realsense_l515/Intel_RealSense_L515.stl" scale="0.001 0.001 0.001"/>
         </geometry>
       </collision>
@@ -41,5 +41,5 @@
     <joint name="camera_depth_joint" type="fixed">
       <origin xyz="0 0 0" rpy="0 0 0"/>
-      <parent link="camera"/>
+      <parent link="camera_link"/>
       <child link="camera_depth_frame" />
     </joint>
@@ -53,5 +53,5 @@
     <joint name="camera_infra_joint" type="fixed">
       <origin xyz="0 ${l515_cam_depth_to_infra_offset} 0" rpy="0 0 0" />
-      <parent link="camera" />
+      <parent link="camera_link"/>
       <child link="camera_infra_frame" />
     </joint>
@@ -65,5 +65,5 @@
     <joint name="camera_color_joint" type="fixed">
       <origin xyz="0 ${l515_cam_depth_to_color_offset} 0" rpy="0 0 0" />
-      <parent link="camera" />
+      <parent link="camera_link" />
       <child link="camera_color_frame" />
     </joint>
@@ -75,6 +75,6 @@
     </joint>
     <link name="camera_color_optical_frame"/>
-    <gazebo reference="camera">
-      <sensor name="camera_rgbd" type="rgbd_camera">
+    <gazebo reference="camera_link">
+      <sensor name="camera" type="rgbd_camera">
         <camera>
           <horizontal_fov>1.5184</horizontal_fov>
@@ -89,5 +89,5 @@
         </camera>
         <always_on>1</always_on>
-        <gz_frame_id>camera</gz_frame_id>
+        <gz_frame_id>camera_link</gz_frame_id>
         <topic>camera</topic>
         <update_rate>5</update_rate>
