Commit message: Tool communication working

File: src/ur_custom/ur_custom_description/urdf/sensors/camera.urdf.xacro (robot description, xacro)
@@ -16,5 +16,5 @@
     <link name="camera">
       <visual>
-        <origin rpy="0 0 0" xyz="0 -0.07 -0.01"/>
+        <origin rpy="0 0 0" xyz="0 -0.07 0"/>
         <geometry>
           <mesh filename="file://$(find ur_custom_description)/meshes/realsense_l515/Intel_RealSense_L515.stl" scale="0.001 0.001 0.001"/>
@@ -25,7 +25,7 @@
       </visual>
       <collision>
-        <origin rpy="0 0 0" xyz="0 -0.07 -0.01"/>
+        <origin rpy="0 0 0" xyz="0 -0.07 0"/>
         <geometry>
-          <mesh filename="file://$(find ur_custom_description)/meshes/realsense_l515/Intel_RealSense_L515.stl" scale="0.0015 0.0015 0.0015"/>
+          <mesh filename="file://$(find ur_custom_description)/meshes/realsense_l515/Intel_RealSense_L515.stl" scale="0.0015 0.0015 0.002"/>
         </geometry>
       </collision>

Commit message: Hardcoded sequence working, approx poses

File: src/ur_custom/ur_custom_description/urdf/sensors/camera.urdf.xacro (robot description, xacro)
@@ -30,4 +30,10 @@
         </geometry>
       </collision>
+      <collision>
+          <origin rpy="0 0 0" xyz="0 0 -0.022"/>
+          <geometry>
+              <cylinder radius="0.06" length="0.05"/>
+          </geometry>
+      </collision>
       <inertial>
         <mass value="0.095" />
