Commit message: Cleaning code

File: src/ur_custom/ur_custom_description/srdf/ur3e_with_gripper_camera.srdf.xacro (robot description, xacro)
@@ -9,5 +9,5 @@
   <!--SUBGROUPS - Groups can also be formed by referencing to already defined group names-->
   <group name="ur_manipulator">
-    <chain base_link="base_link" tip_link="tool0"/>
+    <chain base_link="base_link" tip_link="tool_tip"/>
   </group>
   <!--GROUP STATES - Purpose - Define a named state for a particular group, in terms of joint values. This is useful to define states like 'folded arms'-->
@@ -36,15 +36,4 @@
     <joint name="wrist_3_joint" value="-0.11" />
   </group_state>
-  <!--
-    <joint name="gripper_controller" value="0.019" />
-    <joint name="gripper_base_to_gripper_right" value="0.019" />
-  -->
-  <!--END EFFECTOR - Purpose - Represent information about an end effector.-->
-  <group name="end_effector">
-    <link name="gripper_base" />
-    <link name="gripper_left" />
-    <link name="gripper_right" />
-    <link name="camera" />
-  </group>
   <!--VIRTUAL JOINT - Purpose - this element defines a virtual joint between a robot link and an external frame of reference (considered fixed with respect to the robot)-->
   <!--DISABLE COLLISIONS - By default it is assumed that any link of the robot could potentially come into collision with any other link in the robot. This tag disables collision checking between a specified pair of links. -->
@@ -69,3 +58,11 @@
   <disable_collisions link1="gripper_base" link2="camera" reason="Adjacent" />
   <disable_collisions link1="wrist_2_link" link2="camera" reason="Adjacent" />
+  <disable_collisions link1="gripper_left" link2="camera" reason="Never" />
+  <disable_collisions link1="gripper_right" link2="camera" reason="Never" />
+  <disable_collisions link1="tool_tip" link2="tool0" reason="Never" />
+  <disable_collisions link1="tool_tip" link2="wrist_3_link" reason="Never" />
+  <disable_collisions link1="tool_tip" link2="gripper_base" reason="Adjacent" />
+  <disable_collisions link1="tool_tip" link2="camera" reason="Adjacent" />
+  <disable_collisions link1="tool_tip" link2="gripper_left" reason="Adjacent" />
+  <disable_collisions link1="tool_tip" link2="gripper_right" reason="Adjacent" />
 </robot>

File: src/ur_custom/ur_custom_description/urdf/mech/gripper.urdf.xacro (robot description, xacro)
@@ -31,7 +31,7 @@
       <collision>
         <geometry>
-          <mesh filename="file://$(find ur_custom_description)/meshes/onrobot_2fg7/base_link.stl" scale="0.0012 0.0012 0.001"/>
+          <box size="0.11 0.1 0.16" />
         </geometry>
-        <origin xyz="0 0 0" rpy="0 0 0"/>
+        <origin xyz="0 0 0.08" rpy="0 0 0"/>
       </collision>
     </link>
@@ -59,5 +59,5 @@
       <collision>
         <geometry>
-          <mesh filename="file://$(find ur_custom_description)/meshes/onrobot_2fg7/left_finger_link.stl" scale="0.0013 0.0013 0.001"/>
+          <mesh filename="file://$(find ur_custom_description)/meshes/onrobot_2fg7/left_finger_link.stl" scale="0.001 0.001 0.001"/>
         </geometry>
         <origin xyz="-0.032239 0.029494 -0.12005" rpy="0 0 0"/>
@@ -82,5 +82,5 @@
       <collision>
         <geometry>
-          <mesh filename="file://$(find ur_custom_description)/meshes/onrobot_2fg7/right_finger_link.stl" scale="0.0013 0.0013 0.001"/>
+          <mesh filename="file://$(find ur_custom_description)/meshes/onrobot_2fg7/right_finger_link.stl" scale="0.001 0.001 0.001"/>
         </geometry>
         <origin xyz="0.054361 0.029494 -0.12005" rpy="0 0 0"/>
@@ -97,23 +97,11 @@
       <origin xyz="-0.054361 -0.029494 0.12005" rpy="0 0 0"/>
     </joint>
-    <!--
-    <joint name="${prefix}gripper_controller" type="fixed">
-      <axis xyz="-1 0 0"/>
-      <limit effort="${joint_effort}" lower="0.0" upper="0.019" velocity="${joint_velocity}"/>
-      <parent link="${prefix}gripper_base"/>
-      <child link="${prefix}gripper_left"/>
-      <origin xyz="0.032239 -0.029494 0.12005" rpy="0 0 0"/>
-      <dynamics damping="${joint_damping}" friction="${joint_friction}"/>
+    <link name="tool_tip">
+    </link>
+    <joint name="$tool0_to_tool_tip" type="fixed">
+      <parent link="tool0"/>
+      <child link="tool_tip"/>
+      <origin xyz="0 0 0.16" rpy="0 0 0"/>
     </joint>
-    <joint name="${prefix}gripper_base_to_${prefix}gripper_right" type="fixed">
-      <axis xyz="1 0 0"/>
-      <limit effort="${joint_effort}" lower="-0.019" upper="0.019" velocity="${joint_velocity}"/>
-      <parent link="${prefix}gripper_base"/>
-      <child link="${prefix}gripper_right"/>
-      <origin xyz="-0.054361 -0.029494 0.12005" rpy="0 0 0"/>
-      <mimic joint="${prefix}gripper_controller" multiplier="1.0" offset="0"/>
-      <dynamics damping="${joint_damping}" friction="${joint_friction}"/>
-    </joint>
-    -->
   </xacro:macro>
 </robot>

File: src/ur_custom/ur_custom_description/urdf/sensors/camera.urdf.xacro (robot description, xacro)
@@ -3,10 +3,4 @@
   <xacro:arg name="prefix" default=""/>
   <xacro:arg name="parent" default="tool0"/>
-     <xacro:property name="M_PI" value="3.1415926535897931" />
-     <xacro:property name="l515_cam_width" value="0.061"/>
-     <xacro:property name="l515_cam_height" value="0.061"/>
-     <xacro:property name="l515_cam_depth" value="0.026"/>
-     <xacro:property name="l515_cam_depth_to_infra_offset" value="0.0"/>
-     <xacro:property name="l515_cam_depth_to_color_offset" value="0.012"/>
     <joint name="camera_joint" type="fixed">
       <parent link="$(arg prefix)$(arg parent)"/>
@@ -16,29 +10,33 @@
     <link name="camera">
       <visual>
-        <origin rpy="0 0 0" xyz="0 -0.07 0"/>
+        <origin rpy="0 0 0" xyz="0 -0.07 0.01"/>
         <geometry>
-          <mesh filename="file://$(find ur_custom_description)/meshes/realsense_l515/Intel_RealSense_L515.stl" scale="0.001 0.001 0.001"/>
+          <box size="0.05 0.05 0.05" />
         </geometry>
-        <material name="aluminum">
-          <color rgba="0.5 0.5 0.5 1"/>
+        <material name="silver">
+          <color rgba="0.600 0.600 0.600 1.000"/>
         </material>
       </visual>
       <collision>
-        <origin rpy="0 0 0" xyz="0 -0.07 0"/>
+        <origin rpy="0 0 0" xyz="0 -0.07 0.01"/>
         <geometry>
-          <mesh filename="file://$(find ur_custom_description)/meshes/realsense_l515/Intel_RealSense_L515.stl" scale="0.0015 0.0015 0.002"/>
+          <box size="0.08 0.08 0.08" />
         </geometry>
       </collision>
+      <visual>
+        <origin rpy="0 0 0" xyz="0 0 -0.01"/>
+        <geometry>
+          <cylinder radius="0.04" length="0.015"/>
+        </geometry>
+        <material name="silver">
+          <color rgba="0.600 0.600 0.600 1.000"/>
+        </material>
+      </visual>
       <collision>
-          <origin rpy="0 0 0" xyz="0 0 -0.022"/>
-          <geometry>
-              <cylinder radius="0.06" length="0.05"/>
-          </geometry>
+        <origin rpy="0 0 0" xyz="0 0 -0.01"/>
+        <geometry>
+          <cylinder radius="0.06" length="0.05"/>
+        </geometry>
       </collision>
-      <inertial>
-        <mass value="0.095" />
-        <origin rpy="0 0 0" xyz="0 -0.07 -0.01"/>
-        <inertia ixx="0.000044" ixy="0.0" ixz="0.0" iyy="0.000027" iyz="0.0" izz="0.000027" />
-      </inertial>
     </link>
 </robot>
